Commit message: revert messed up xacro file

File: yumi_description/urdf/yumi.urdf.xacro (robot description, xacro)
@@ -1,857 +1,41 @@
-<?xml version="1.0" ?>
-<!-- =================================================================================== -->
-<!-- |    This document was autogenerated by xacro from yumi.urdf                      | -->
-<!-- |    EDITING THIS FILE BY HAND IS NOT RECOMMENDED                                 | -->
-<!-- =================================================================================== -->
-<!-- =================================================================================== -->
-<!-- |    This document was autogenerated by xacro from yumi.urdf.xacro                | -->
-<!-- |    EDITING THIS FILE BY HAND IS NOT RECOMMENDED                                 | -->
-<!-- =================================================================================== -->
-<robot name="yumi">
-  <material name="Black">
-    <color rgba="0.0 0.0 0.0 1.0"/>
-  </material>
-  <material name="Blue">
-    <color rgba="0.0 0.0 0.8 1.0"/>
-  </material>
-  <material name="Green">
-    <color rgba="0.0 0.8 0.0 1.0"/>
-  </material>
-  <material name="Grey">
-    <color rgba="0.5 0.5 0.5 1.0"/>
-  </material>
-  <material name="Light_Grey">
-    <color rgba="0.8 0.8 0.8 1.0"/>
-  </material>
-  <material name="Ivory">
-    <color rgba="1.0 1.0 0.94 1.0"/>
-  </material>
-  <material name="Orange">
-    <color rgba="1.0 0.4235294117647059 0.0392156862745098 1.0"/>
-  </material>
-  <material name="Brown">
-    <color rgba="0.8705882352941177 0.8117647058823529 0.7647058823529411 1.0"/>
-  </material>
-  <material name="Red">
-    <color rgba="0.8 0.0 0.0 1.0"/>
-  </material>
-  <material name="White">
-    <color rgba="1.0 1.0 1.0 1.0"/>
-  </material>
-  <gazebo>
-    <plugin filename="libgazebo_ros_control.so" name="gazebo_ros_controller">
-      <robotNamespace>/yumi</robotNamespace>
-    </plugin>
-  </gazebo>
-  <link name="yumi_base_link"/>
-  <joint name="yumi_base_link_to_body" type="fixed">
-    <parent link="yumi_base_link"/>
-    <child link="yumi_body"/>
-    <origin rpy="0 0 0" xyz="0 0 0"/>
-  </joint>
-  <link name="yumi_body">
-    <inertial>
-      <origin rpy="0 0 0" xyz="0 0 0"/>
-      <mass value="15"/>
-      <inertia ixx="0.5" ixy="0" ixz="0" iyy="0.6" iyz="0" izz="0.3"/>
-    </inertial>
-    <visual>
-      <origin rpy="0 0 0" xyz="0 0 0"/>
-      <geometry>
-        <mesh filename="package://yumi_description/meshes/body.stl"/>
-      </geometry>
-      <material name="Light_Grey"/>
-    </visual>
-    <collision>
-      <origin rpy="0 0 0" xyz="0 0 0"/>
-      <geometry>
-        <mesh filename="package://yumi_description/meshes/coarse/body.stl"/>
-      </geometry>
-      <material name="Light_Grey"/>
-    </collision>
-  </link>
-  <!--///////////////////////////////////// RIGHT ARM ////////////////////////////////  -->
-  <!-- joint between body and link_1_r -->
-  <joint name="yumi_robr_joint_1" type="revolute">
-    <parent link="yumi_body"/>
-    <child link="yumi_link_1_r"/>
-    <origin rpy="-0.9795   -0.5682   -2.3155" xyz="0.05355 -0.0725 0.41492"/>
-    <axis xyz="0 0 1"/>
-    <limit effort="300" lower="-2.940879789610445" upper="2.940879789610445" velocity="3.141592653589793"/>
-    <dynamics damping="0.5"/>
-  </joint>
-  <link name="yumi_link_1_r">
-    <inertial>
-      <origin rpy="0 0 0" xyz="0 -0.03 0.12"/>
-      <mass value="2"/>
-      <inertia ixx="0.1" ixy="0" ixz="0" iyy="0.1" iyz="0" izz="0.1"/>
-    </inertial>
-    <visual>
-      <origin rpy="0 0 0" xyz="0 0 0"/>
-      <geometry>
-        <mesh filename="package://yumi_description/meshes/link_1.stl"/>
-      </geometry>
-      <material name="Grey"/>
-    </visual>
-    <collision>
-      <origin rpy="0 0 0" xyz="0 0 0"/>
-      <geometry>
-        <mesh filename="package://yumi_description/meshes/coarse/link_1.stl"/>
-      </geometry>
-      <material name="Grey"/>
-    </collision>
-  </link>
-  <!-- joint between link_1_r and link_2_r -->
-  <joint name="yumi_robr_joint_2" type="revolute">
-    <parent link="yumi_link_1_r"/>
-    <child link="yumi_link_2_r"/>
-    <origin rpy="1.5707963267948966 0.0 0.0" xyz="0.03 0.0 0.1"/>
-    <axis xyz="0 0 1"/>
-    <limit effort="300" lower="-2.504547476611863" upper="0.7592182246175333" velocity="3.141592653589793"/>
-    <dynamics damping="0.5"/>
-  </joint>
-  <link name="yumi_link_2_r">
-    <inertial>
-      <origin rpy="0 0 0" xyz="0 0 0"/>
-      <mass value="2"/>
-      <inertia ixx="0.1" ixy="0" ixz="0" iyy="0.1" iyz="0" izz="0.1"/>
-    </inertial>
-    <visual>
-      <origin rpy="0 0 0" xyz="0 0 0"/>
-      <geometry>
-        <mesh filename="package://yumi_description/meshes/link_2.stl"/>
-      </geometry>
-      <material name="Grey"/>
-    </visual>
-    <collision>
-      <origin rpy="0 0 0" xyz="0 0 0"/>
-      <geometry>
-        <mesh filename="package://yumi_description/meshes/coarse/link_2.stl"/>
-      </geometry>
-      <material name="Grey"/>
-    </collision>
-  </link>
-  <!-- joint between link_2_r and link_3_r -->
-  <joint name="yumi_robr_joint_7" type="revolute">
-    <parent link="yumi_link_2_r"/>
-    <child link="yumi_link_3_r"/>
-    <origin rpy="-1.5707963267948966 0.0 0.0" xyz="-0.03 0.17283 0.0"/>
-    <axis xyz="0 0 1"/>
-    <limit effort="300" lower="-2.940879789610445" upper="2.940879789610445" velocity="3.141592653589793"/>
-    <dynamics damping="0.5"/>
-  </joint>
-  <link name="yumi_link_3_r">
-    <inertial>
-      <origin rpy="0 0 0" xyz="0 0 0"/>
-      <mass value="2"/>
-      <inertia ixx="0.1" ixy="0" ixz="0" iyy="0.1" iyz="0" izz="0.1"/>
-    </inertial>
-    <visual>
-      <origin rpy="0 0 0" xyz="0 0 0"/>
-      <geometry>
-        <mesh filename="package://yumi_description/meshes/link_3.stl"/>
-      </geometry>
-      <material name="Grey"/>
-    </visual>
-    <collision>
-      <origin rpy="0 0 0" xyz="0 0 0"/>
-      <geometry>
-        <mesh filename="package://yumi_description/meshes/coarse/link_3.stl"/>
-      </geometry>
-      <material name="Grey"/>
-    </collision>
-  </link>
-  <!-- joint between link_3_r and link_4_r -->
-  <joint name="yumi_robr_joint_3" type="revolute">
-    <parent link="yumi_link_3_r"/>
-    <child link="yumi_link_4_r"/>
-    <origin rpy="1.5707963267948966 -1.5707963267948966 0.0" xyz="-0.04188 0.0 0.07873"/>
-    <axis xyz="0 0 1"/>
-    <limit effort="300" lower="-2.155481626212997" upper="1.3962634015954636" velocity="3.141592653589793"/>
-    <dynamics damping="0.5"/>
-  </joint>
-  <link name="yumi_link_4_r">
-    <inertial>
-      <origin rpy="0 0 0" xyz="0 0 0"/>
-      <mass value="2"/>
-      <inertia ixx="0.1" ixy="0" ixz="0" iyy="0.1" iyz="0" izz="0.1"/>
-    </inertial>
-    <visual>
-      <origin rpy="0 0 0" xyz="0 0 0"/>
-      <geometry>
-        <mesh filename="package://yumi_description/meshes/link_4.stl"/>
-      </geometry>
-      <material name="Grey"/>
-    </visual>
-    <collision>
-      <origin rpy="0 0 0" xyz="0 0 0"/>
-      <geometry>
-        <mesh filename="package://yumi_description/meshes/coarse/link_4.stl"/>
-      </geometry>
-      <material name="Grey"/>
-    </collision>
-  </link>
-  <!-- joint between link_4_r and link_5_r -->
-  <joint name="yumi_robr_joint_4" type="revolute">
-    <parent link="yumi_link_4_r"/>
-    <child link="yumi_link_5_r"/>
-    <origin rpy="-1.5707963267948966 0.0 0.0" xyz="0.0405 0.16461 0.0"/>
-    <axis xyz="0 0 1"/>
-    <limit effort="300" lower="-5.061454830783555" upper="5.061454830783555" velocity="6.981317007977318"/>
-    <dynamics damping="0.5"/>
-  </joint>
-  <link name="yumi_link_5_r">
-    <inertial>
-      <origin rpy="0 0 0" xyz="0 0 0"/>
-      <mass value="2"/>
-      <inertia ixx="0.1" ixy="0" ixz="0" iyy="0.1" iyz="0" izz="0.1"/>
-    </inertial>
-    <visual>
-      <origin rpy="0 0 0" xyz="0 0 0"/>
-      <geometry>
-        <mesh filename="package://yumi_description/meshes/link_5.stl"/>
-      </geometry>
-      <material name="Grey"/>
-    </visual>
-    <collision>
-      <origin rpy="0 0 0" xyz="0 0 0"/>
-      <geometry>
-        <mesh filename="package://yumi_description/meshes/coarse/link_5.stl"/>
-      </geometry>
-      <material name="Grey"/>
-    </collision>
-  </link>
-  <!-- joint between link_5_r and link_6_r -->
-  <joint name="yumi_robr_joint_5" type="revolute">
-    <parent link="yumi_link_5_r"/>
-    <child link="yumi_link_6_r"/>
-    <origin rpy="1.5707963267948966 0.0 0.0" xyz="-0.027 0 0.10039"/>
-    <axis xyz="0 0 1"/>
-    <limit effort="300" lower="-1.53588974175501" upper="2.4085543677521746" velocity="6.981317007977318"/>
-    <dynamics damping="0.5"/>
-  </joint>
-  <link name="yumi_link_6_r">
-    <inertial>
-      <origin rpy="0 0 0" xyz="0 0 0"/>
-      <mass value="2"/>
-      <inertia ixx="0.1" ixy="0" ixz="0" iyy="0.1" iyz="0" izz="0.1"/>
-    </inertial>
-    <visual>
-      <origin rpy="0 0 0" xyz="0 0 0"/>
-      <geometry>
-        <mesh filename="package://yumi_description/meshes/link_6.stl"/>
-      </geometry>
-      <material name="Grey"/>
-    </visual>
-    <collision>
-      <origin rpy="0 0 0" xyz="0 0 0"/>
-      <geometry>
-        <mesh filename="package://yumi_description/meshes/coarse/link_6.stl"/>
-      </geometry>
-      <material name="Grey"/>
-    </collision>
-  </link>
-  <!-- joint between link_6_r and link_7_r -->
-  <joint name="yumi_robr_joint_6" type="revolute">
-    <parent link="yumi_link_6_r"/>
-    <child link="yumi_link_7_r"/>
-    <origin rpy="-1.5707963267948966 0.0 0.0" xyz="0.027 0.029 0.0"/>
-    <axis xyz="0 0 1"/>
-    <limit effort="300" lower="-3.9968039870670142" upper="3.9968039870670142" velocity="6.981317007977318"/>
-    <dynamics damping="0.5"/>
-  </joint>
-  <link name="yumi_link_7_r">
-    <inertial>
-      <origin rpy="0 0 0" xyz="0 0 0"/>
-      <mass value="2"/>
-      <inertia ixx="0.1" ixy="0" ixz="0" iyy="0.1" iyz="0" izz="0.1"/>
-    </inertial>
-    <visual>
-      <origin rpy="0 0 0" xyz="0 0 0"/>
-      <geometry>
-        <mesh filename="package://yumi_description/meshes/link_7.stl"/>
-      </geometry>
-      <material name="Grey"/>
-    </visual>
-    <collision>
-      <origin rpy="0 0 0" xyz="0 0 0"/>
-      <geometry>
-        <mesh filename="package://yumi_description/meshes/coarse/link_7.stl"/>
-      </geometry>
-      <material name="Grey"/>
-    </collision>
-  </link>
-  <!--///////////////////////////////////// LEFT ARM ////////////////////////////////  -->
-  <!-- joint between body and link_1_l -->
-  <joint name="yumi_robl_joint_1" type="revolute">
-    <parent link="yumi_body"/>
-    <child link="yumi_link_1_l"/>
-    <origin rpy="0.9781 -0.5716 2.3180" xyz="0.05355 0.07250 0.41492"/>
-    <axis xyz="0 0 1"/>
-    <limit effort="300" lower="-2.940879789610445" upper="2.940879789610445" velocity="3.141592653589793"/>
-    <dynamics damping="0.5"/>
-  </joint>
-  <link name="yumi_link_1_l">
-    <inertial>
-      <origin rpy="0 0 0" xyz="0 -0.03 0.12"/>
-      <mass value="2"/>
-      <inertia ixx="0.1" ixy="0" ixz="0" iyy="0.1" iyz="0" izz="0.1"/>
-    </inertial>
-    <visual>
-      <origin rpy="0 0 0" xyz="0 0 0"/>
-      <geometry>
-        <mesh filename="package://yumi_description/meshes/link_1.stl"/>
-      </geometry>
-      <material name="Grey"/>
-    </visual>
-    <collision>
-      <origin rpy="0 0 0" xyz="0 0 0"/>
-      <geometry>
-        <mesh filename="package://yumi_description/meshes/coarse/link_1.stl"/>
-      </geometry>
-      <material name="Grey"/>
-    </collision>
-  </link>
-  <!-- joint between link_1_l and link_2_l -->
-  <joint name="yumi_robl_joint_2" type="revolute">
-    <parent link="yumi_link_1_l"/>
-    <child link="yumi_link_2_l"/>
-    <origin rpy="1.5707963267948966 0.0 0.0" xyz="0.03 0.0 0.1"/>
-    <axis xyz="0 0 1"/>
-    <limit effort="300" lower="-2.504547476611863" upper="0.7592182246175333" velocity="3.141592653589793"/>
-    <dynamics damping="0.5"/>
-  </joint>
-  <link name="yumi_link_2_l">
-    <inertial>
-      <origin rpy="0 0 0" xyz="0 0 0"/>
-      <mass value="2"/>
-      <inertia ixx="0.1" ixy="0" ixz="0" iyy="0.1" iyz="0" izz="0.1"/>
-    </inertial>
-    <visual>
-      <origin rpy="0 0 0" xyz="0 0 0"/>
-      <geometry>
-        <mesh filename="package://yumi_description/meshes/link_2.stl"/>
-      </geometry>
-      <material name="Grey"/>
-    </visual>
-    <collision>
-      <origin rpy="0 0 0" xyz="0 0 0"/>
-      <geometry>
-        <mesh filename="package://yumi_description/meshes/coarse/link_2.stl"/>
-      </geometry>
-      <material name="Grey"/>
-    </collision>
-  </link>
-  <!-- joint between link_2_l and link_3_l -->
-  <joint name="yumi_robl_joint_7" type="revolute">
-    <parent link="yumi_link_2_l"/>
-    <child link="yumi_link_3_l"/>
-    <origin rpy="-1.5707963267948966 0.0 0.0" xyz="-0.03 0.17283 0.0"/>
-    <axis xyz="0 0 1"/>
-    <limit effort="300" lower="-2.940879789610445" upper="2.940879789610445" velocity="3.141592653589793"/>
-    <dynamics damping="0.5"/>
-  </joint>
-  <link name="yumi_link_3_l">
-    <inertial>
-      <origin rpy="0 0 0" xyz="0 0 0"/>
-      <mass value="2"/>
-      <inertia ixx="0.1" ixy="0" ixz="0" iyy="0.1" iyz="0" izz="0.1"/>
-    </inertial>
-    <visual>
-      <origin rpy="0 0 0" xyz="0 0 0"/>
-      <geometry>
-        <mesh filename="package://yumi_description/meshes/link_3.stl"/>
-      </geometry>
-      <material name="Grey"/>
-    </visual>
-    <collision>
-      <origin rpy="0 0 0" xyz="0 0 0"/>
-      <geometry>
-        <mesh filename="package://yumi_description/meshes/coarse/link_3.stl"/>
-      </geometry>
-      <material name="Grey"/>
-    </collision>
-  </link>
-  <!-- joint between link_3_l and link_4_l -->
-  <joint name="yumi_robl_joint_3" type="revolute">
-    <parent link="yumi_link_3_l"/>
-    <child link="yumi_link_4_l"/>
-    <origin rpy="1.5707963267948966 -1.5707963267948966 0.0" xyz="-0.04188 0.0 0.07873"/>
-    <axis xyz="0 0 1"/>
-    <limit effort="300" lower="-2.155481626212997" upper="1.3962634015954636" velocity="3.141592653589793"/>
-    <dynamics damping="0.5"/>
-  </joint>
-  <link name="yumi_link_4_l">
-    <inertial>
-      <origin rpy="0 0 0" xyz="0 0 0"/>
-      <mass value="2"/>
-      <inertia ixx="0.1" ixy="0" ixz="0" iyy="0.1" iyz="0" izz="0.1"/>
-    </inertial>
-    <visual>
-      <origin rpy="0 0 0" xyz="0 0 0"/>
-      <geometry>
-        <mesh filename="package://yumi_description/meshes/link_4.stl"/>
-      </geometry>
-      <material name="Grey"/>
-    </visual>
-    <collision>
-      <origin rpy="0 0 0" xyz="0 0 0"/>
-      <geometry>
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
Commit message: a xacro that actually works

File: yumi_description/urdf/yumi.urdf.xacro (robot description, xacro)
@@ -11,8 +11,9 @@
   <!-- Import Gazebo plugins -->
   <xacro:include filename="$(find yumi_description)/urdf/Gazebo/gazebo.urdf.xacro"/>
+  <!--yumi-->
+  <xacro:arg name="arms_interface" default="VelocityJointInterface"/>
+  <xacro:arg name="grippers_interface" default="EffortJointInterface"/>
+  <xacro:arg name="yumi_setup" default="default"/>
   <xacro:property name="yumi_setup" value="$(arg yumi_setup)" />
-  <xacro:if value="${yumi_setup == 'robot_centric'}">
-  	<!-- Pure YuMi URDF, with no joints connecting it to any other robot or pedestal. Neither accessories. -->
-  </xacro:if>
   <xacro:if value="${yumi_setup == 'default'}">
     <xacro:property name="yumi_parent" value="world" />
@@ -24,8 +25,8 @@
     </joint>
   </xacro:if>
-  <!--yumi-->
-  <xacro:arg name="arms_interface" default="VelocityJointInterface"/>
+  <xacro:if value="${yumi_setup == 'robot_centric'}">
+  	<!-- Pure YuMi URDF, with no joints connecting it to any other robot or pedestal. Neither accessories. -->
+  </xacro:if>
 	  <!-- <xacro:property name="yumi_parent" value="yumi_pedestal" /> -->
-  <xacro:property name="yumi_parent" value="world" />
   <xacro:yumi name="yumi" hardware_interface="hardware_interface/$(arg arms_interface)" parent="${yumi_parent}" >
     <origin xyz="0 0 0.1" rpy="0 0 0" />
