Commit message: rename all joints to abb_robot_driver convention

File: yumi_description/urdf/yumi.urdf (robot description, URDF)
Before this commit: robot yumi, 22 links, 21 joints
Links:
- link gripper_l_finger_l: mass 0.01 -> 0.04
- link gripper_l_finger_r: mass 0.01 -> 0.04
- link gripper_r_finger_l: mass 0.01 -> 0.04
- link gripper_r_finger_r: mass 0.01 -> 0.04
Joints:
- removed joint yumi_joint_1_l
- removed joint yumi_joint_1_r
- removed joint yumi_joint_2_l
- removed joint yumi_joint_2_r
- removed joint yumi_joint_3_l
- removed joint yumi_joint_3_r
- removed joint yumi_joint_4_l
- removed joint yumi_joint_4_r
- removed joint yumi_joint_5_l
- removed joint yumi_joint_5_r
- removed joint yumi_joint_6_l
- removed joint yumi_joint_6_r
- removed joint yumi_joint_7_l
- removed joint yumi_joint_7_r
- added joint yumi_robl_joint_1: type revolute, parent yumi_body, child yumi_link_1_l, origin xyz=0.05355 0.07250 0.41492 rpy=0.9781 -0.5716 2.3180, axis 0 0 1, limit lower=-2.940879789610445 upper=2.940879789610445 effort=300 velocity=3.141592653589793
- added joint yumi_robl_joint_2: type revolute, parent yumi_link_1_l, child yumi_link_2_l, origin xyz=0.03 0.0 0.1 rpy=1.5707963267948966 0.0 0.0, axis 0 0 1, limit lower=-2.504547476611863 upper=0.7592182246175333 effort=300 velocity=3.141592653589793
- added joint yumi_robl_joint_3: type revolute, parent yumi_link_3_l, child yumi_link_4_l, origin xyz=-0.04188 0.0 0.07873 rpy=1.5707963267948966 -1.5707963267948966 0.0, axis 0 0 1, limit lower=-2.155481626212997 upper=1.3962634015954636 effort=300 velocity=3.141592653589793
- added joint yumi_robl_joint_4: type revolute, parent yumi_link_4_l, child yumi_link_5_l, origin xyz=0.0405 0.16461 0.0 rpy=-1.5707963267948966 0.0 0.0, axis 0 0 1, limit lower=-5.061454830783555 upper=5.061454830783555 effort=300 velocity=6.981317007977318
- added joint yumi_robl_joint_5: type revolute, parent yumi_link_5_l, child yumi_link_6_l, origin xyz=-0.027 0 0.10039 rpy=1.5707963267948966 0.0 0.0, axis 0 0 1, limit lower=-1.53588974175501 upper=2.4085543677521746 effort=300 velocity=6.981317007977318
- added joint yumi_robl_joint_6: type revolute, parent yumi_link_6_l, child yumi_link_7_l, origin xyz=0.027 0.029 0.0 rpy=-1.5707963267948966 0.0 0.0, axis 0 0 1, limit lower=-3.9968039870670142 upper=3.9968039870670142 effort=300 velocity=6.981317007977318
- added joint yumi_robl_joint_7: type revolute, parent yumi_link_2_l, child yumi_link_3_l, origin xyz=-0.03 0.17283 0.0 rpy=-1.5707963267948966 0.0 0.0, axis 0 0 1, limit lower=-2.940879789610445 upper=2.940879789610445 effort=300 velocity=3.141592653589793
- added joint yumi_robr_joint_1: type revolute, parent yumi_body, child yumi_link_1_r, origin xyz=0.05355 -0.0725 0.41492 rpy=-0.9795   -0.5682   -2.3155, axis 0 0 1, limit lower=-2.940879789610445 upper=2.940879789610445 effort=300 velocity=3.141592653589793
- added joint yumi_robr_joint_2: type revolute, parent yumi_link_1_r, child yumi_link_2_r, origin xyz=0.03 0.0 0.1 rpy=1.5707963267948966 0.0 0.0, axis 0 0 1, limit lower=-2.504547476611863 upper=0.7592182246175333 effort=300 velocity=3.141592653589793
- added joint yumi_robr_joint_3: type revolute, parent yumi_link_3_r, child yumi_link_4_r, origin xyz=-0.04188 0.0 0.07873 rpy=1.5707963267948966 -1.5707963267948966 0.0, axis 0 0 1, limit lower=-2.155481626212997 upper=1.3962634015954636 effort=300 velocity=3.141592653589793
- added joint yumi_robr_joint_4: type revolute, parent yumi_link_4_r, child yumi_link_5_r, origin xyz=0.0405 0.16461 0.0 rpy=-1.5707963267948966 0.0 0.0, axis 0 0 1, limit lower=-5.061454830783555 upper=5.061454830783555 effort=300 velocity=6.981317007977318
- added joint yumi_robr_joint_5: type revolute, parent yumi_link_5_r, child yumi_link_6_r, origin xyz=-0.027 0 0.10039 rpy=1.5707963267948966 0.0 0.0, axis 0 0 1, limit lower=-1.53588974175501 upper=2.4085543677521746 effort=300 velocity=6.981317007977318
- added joint yumi_robr_joint_6: type revolute, parent yumi_link_6_r, child yumi_link_7_r, origin xyz=0.027 0.029 0.0 rpy=-1.5707963267948966 0.0 0.0, axis 0 0 1, limit lower=-3.9968039870670142 upper=3.9968039870670142 effort=300 velocity=6.981317007977318
- added joint yumi_robr_joint_7: type revolute, parent yumi_link_2_r, child yumi_link_3_r, origin xyz=-0.03 0.17283 0.0 rpy=-1.5707963267948966 0.0 0.0, axis 0 0 1, limit lower=-2.940879789610445 upper=2.940879789610445 effort=300 velocity=3.141592653589793
- joint gripper_l_joint_m: origin xyz=0 0.0065 0.0837 rpy=0 0 3.14159265359 -> xyz=0 0.0065 0.0837 rpy=0 0 3.141592653589793
- joint gripper_r_joint_m: origin xyz=0 0.0065 0.0837 rpy=0 0 3.14159265359 -> xyz=0 0.0065 0.0837 rpy=0 0 3.141592653589793
- joint yumi_link_7_l_joint: origin xyz=0 0 0.007 rpy=0 0 3.14159265359 -> xyz=0 0 0.007 rpy=0 0 3.141592653589793
- joint yumi_link_7_r_joint: origin xyz=0 0 0.007 rpy=0 0 3.14159265359 -> xyz=0 0 0.007 rpy=0 0 3.141592653589793

File: yumi_description/urdf/yumi.urdf.xacro (robot description, xacro)
@@ -12,4 +12,7 @@
   <xacro:include filename="$(find yumi_description)/urdf/Gazebo/gazebo.urdf.xacro"/>
   <!--yumi-->
+  <xacro:arg name="arms_interface" default="VelocityJointInterface"/>
+	  <!-- <xacro:property name="yumi_parent" value="yumi_pedestal" /> -->
+  <xacro:property name="yumi_parent" value="world" />
   <xacro:yumi name="yumi" hardware_interface="hardware_interface/$(arg arms_interface)" parent="${yumi_parent}" >
     <origin xyz="0 0 0.1" rpy="0 0 0" />

File: yumi_description/urdf/yumi.xacro (robot description, xacro)
@@ -38,5 +38,5 @@
    <!--///////////////////////////////////// RIGHT ARM ////////////////////////////////  -->
    <!-- joint between body and link_1_r -->
-    <joint name="${name}_joint_1_r" type="revolute">
+    <joint name="${name}_robr_joint_1" type="revolute">
       <parent link="${name}_body"/>
       <child link="${name}_link_1_r"/>
@@ -69,5 +69,5 @@
     </link>
    <!-- joint between link_1_r and link_2_r -->
-    <joint name="${name}_joint_2_r" type="revolute">
+    <joint name="${name}_robr_joint_2" type="revolute">
       <parent link="${name}_link_1_r"/>
       <child link="${name}_link_2_r"/>
@@ -100,5 +100,5 @@
     </link>
      <!-- joint between link_2_r and link_3_r -->
-      <joint name="${name}_joint_7_r" type="revolute">
+      <joint name="${name}_robr_joint_7" type="revolute">
         <parent link="${name}_link_2_r"/>
         <child link="${name}_link_3_r"/>
@@ -131,5 +131,5 @@
     </link>
     <!-- joint between link_3_r and link_4_r -->
-    <joint name="${name}_joint_3_r" type="revolute">
+    <joint name="${name}_robr_joint_3" type="revolute">
       <parent link="${name}_link_3_r"/>
       <child link="${name}_link_4_r"/>
@@ -162,5 +162,5 @@
     </link>
     <!-- joint between link_4_r and link_5_r -->
-    <joint name="${name}_joint_4_r" type="revolute">
+    <joint name="${name}_robr_joint_4" type="revolute">
       <parent link="${name}_link_4_r"/>
       <child link="${name}_link_5_r"/>
@@ -193,5 +193,5 @@
     </link>
     <!-- joint between link_5_r and link_6_r -->
-    <joint name="${name}_joint_5_r" type="revolute">
+    <joint name="${name}_robr_joint_5" type="revolute">
       <parent link="${name}_link_5_r"/>
       <child link="${name}_link_6_r"/>
@@ -224,5 +224,5 @@
     </link>
     <!-- joint between link_6_r and link_7_r -->
-    <joint name="${name}_joint_6_r" type="revolute">
+    <joint name="${name}_robr_joint_6" type="revolute">
       <parent link="${name}_link_6_r"/>
       <child link="${name}_link_7_r"/>
@@ -256,5 +256,5 @@
     <!--///////////////////////////////////// LEFT ARM ////////////////////////////////  -->
     <!-- joint between body and link_1_l -->
-    <joint name="${name}_joint_1_l" type="revolute">
+    <joint name="${name}_robl_joint_1" type="revolute">
       <parent link="${name}_body"/>
       <child link="${name}_link_1_l"/>
@@ -287,5 +287,5 @@
     </link>
     <!-- joint between link_1_l and link_2_l -->
-    <joint name="${name}_joint_2_l" type="revolute">
+    <joint name="${name}_robl_joint_2" type="revolute">
       <parent link="${name}_link_1_l"/>
       <child link="${name}_link_2_l"/>
@@ -318,5 +318,5 @@
     </link>
     <!-- joint between link_2_l and link_3_l -->
-    <joint name="${name}_joint_7_l" type="revolute">
+    <joint name="${name}_robl_joint_7" type="revolute">
       <parent link="${name}_link_2_l"/>
       <child link="${name}_link_3_l"/>
@@ -349,5 +349,5 @@
     </link>
     <!-- joint between link_3_l and link_4_l -->
-    <joint name="${name}_joint_3_l" type="revolute">
+    <joint name="${name}_robl_joint_3" type="revolute">
       <parent link="${name}_link_3_l"/>
       <child link="${name}_link_4_l"/>
@@ -380,5 +380,5 @@
     </link>
     <!-- joint between link_4_l and link_5_l -->
-    <joint name="${name}_joint_4_l" type="revolute">
+    <joint name="${name}_robl_joint_4" type="revolute">
       <parent link="${name}_link_4_l"/>
       <child link="${name}_link_5_l"/>
@@ -411,5 +411,5 @@
     </link>
     <!-- joint between link_5_l and link_6_l -->
-    <joint name="${name}_joint_5_l" type="revolute">
+    <joint name="${name}_robl_joint_5" type="revolute">
       <parent link="${name}_link_5_l"/>
       <child link="${name}_link_6_l"/>
@@ -442,5 +442,5 @@
     </link>
     <!-- joint between link_6_l and link_7_l -->
-    <joint name="${name}_joint_6_l" type="revolute">
+    <joint name="${name}_robl_joint_6" type="revolute">
       <parent link="${name}_link_6_l"/>
       <child link="${name}_link_7_l"/>
